Commit message: marco: fixed configurations

File: planar_cartesian_robot_description/urdf/cartesian_cell.xacro (robot description, xacro)
@@ -6,5 +6,5 @@
     <parent link="world"/>
     <child link="link_Z"/>
-    <origin xyz="0 0 0.5"/>
+    <origin xyz="0 0 0" />
   </joint>
 </robot>

File: planar_cartesian_robot_description/urdf/cartesian_robot.urdf.xacro (robot description, xacro)
@@ -36,6 +36,6 @@
     <child link="link_X"/>
     <axis xyz = "0 0 1" />
-    <origin rpy="0 0 0" xyz="0.5 0 -0.5"/>
-    <limit effort="1000.0" lower="0" upper="1" velocity="0.5"/>
+    <origin rpy="0 0 0" xyz="0.5 0 0.0"/>
+    <limit effort="1000.0" lower="-1" upper="1" velocity="0.5"/>
   </joint>
   <joint name="from_X_to_fake" type="prismatic">
@@ -44,5 +44,5 @@
     <axis xyz = "1 0 0" />
     <origin rpy="0 0 0" xyz="-0.5 0 0"/>
-    <limit effort="1000.0" lower="0" upper="1" velocity="0.5"/>
+    <limit effort="1000.0" lower="-1" upper="1" velocity="0.5"/>
   </joint>
   <joint name="from_fake_to_Y" type="prismatic">
@@ -51,5 +51,5 @@
     <axis xyz = "0 1 0" />
     <origin rpy="0 0 0" xyz="0 -0.5 0"/>
-    <limit effort="1000.0" lower="0" upper="1" velocity="0.5"/>
+    <limit effort="1000.0" lower="-1" upper="1" velocity="0.5"/>
   </joint>
   <joint name="from_Y_to_end" type="fixed">
