Commit message: changes to benchmark

File: planar_cartesian_robot_description/urdf/cartesian_robot.urdf.xacro (robot description, xacro)
@@ -41,5 +41,5 @@
     <visual>
       <geometry>
-        <sphere radius="0.005"/>
+        <sphere radius="0.015"/>
       </geometry>
       <origin rpy="0 0 0" xyz="0 0 0"/>
@@ -49,5 +49,5 @@
       <origin rpy="0 0 0" xyz="0 0 0"/>
       <geometry>
-        <sphere radius="0.025"/>
+        <sphere radius="0.015"/>
       </geometry>
     </collision>

Commit message: fixed urdf robot structure and regenerated moveit_config

File: planar_cartesian_robot_description/urdf/cartesian_robot.urdf.xacro (robot description, xacro)
@@ -14,28 +14,7 @@
   </material>
   <link name="link_Z"/>
+  <link name="link_X"/>
   <link name="link_Y"/>
-  <joint name="from_Z_to_Y" type="fixed">
-    <parent link="link_Z"/>
-    <child link="link_Y"/>
-    <axis xyz = "0 0 1" />
-    <origin rpy="0 0 0" xyz="0 0.5 -0.5"/>
-    <limit effort="1000.0" lower="0" upper="1" velocity="0.5"/>
-  </joint>
   <link name="link_fake"/>
-  <joint name="from_Y_to_fake" type="prismatic">
-    <parent link="link_Y"/>
-    <child link="link_fake"/>
-    <axis xyz = "0 1 0" />
-    <origin rpy="0 0 0" xyz="0 -0.5 0"/>
-    <limit effort="1000.0" lower="0" upper="1" velocity="0.5"/>
-  </joint>
-  <link name="link_X"/>
-  <joint name="from_fake_to_X" type="prismatic">
-    <parent link="link_fake"/>
-    <child link="link_X"/>
-    <axis xyz = "1 0 0" />
-    <origin rpy="0 0 0" xyz="-0.5 0 0"/>
-    <limit effort="1000.0" lower="0" upper="1" velocity="0.5"/>
-  </joint>
   <link name="end_effector">
     <visual>
@@ -53,8 +32,29 @@
     </collision>
   </link>
-  <joint name="from_X_to_end" type="fixed">
+  <joint name="from_Z_to_X" type="fixed">
+    <parent link="link_Z"/>
+    <child link="link_X"/>
+    <axis xyz = "0 0 1" />
+    <origin rpy="0 0 0" xyz="0.5 0 -0.5"/>
+    <limit effort="1000.0" lower="0" upper="1" velocity="0.5"/>
+  </joint>
+  <joint name="from_X_to_fake" type="prismatic">
     <parent link="link_X"/>
+    <child link="link_fake"/>
+    <axis xyz = "1 0 0" />
+    <origin rpy="0 0 0" xyz="-0.5 0 0"/>
+    <limit effort="1000.0" lower="0" upper="1" velocity="0.5"/>
+  </joint>
+  <joint name="from_fake_to_Y" type="prismatic">
+    <parent link="link_fake"/>
+    <child link="link_Y"/>
+    <axis xyz = "0 1 0" />
+    <origin rpy="0 0 0" xyz="0 -0.5 0"/>
+    <limit effort="1000.0" lower="0" upper="1" velocity="0.5"/>
+  </joint>
+  <joint name="from_Y_to_end" type="fixed">
+    <parent link="link_Y"/>
     <child link="end_effector"/>
-    <origin rpy="0 0 0" xyz="0.5 0 0"/>
+    <origin rpy="0 0 0" xyz="0 0.5 0"/>
   </joint>
 </robot>

Commit message: marco: changed position bounds to 0-1

File: planar_cartesian_robot_description/urdf/cartesian_robot.urdf.xacro (robot description, xacro)
@@ -37,5 +37,5 @@
     <axis xyz = "0 0 1" />
     <origin rpy="0 0 0" xyz="0.5 0 0.0"/>
-    <limit effort="1000.0" lower="-1" upper="1" velocity="0.5"/>
+    <limit effort="1000.0" lower="0" upper="1" velocity="0.5"/>
   </joint>
   <joint name="from_X_to_fake" type="prismatic">
@@ -44,5 +44,5 @@
     <axis xyz = "1 0 0" />
     <origin rpy="0 0 0" xyz="-0.5 0 0"/>
-    <limit effort="1000.0" lower="-1" upper="1" velocity="0.5"/>
+    <limit effort="1000.0" lower="0" upper="1" velocity="0.5"/>
   </joint>
   <joint name="from_fake_to_Y" type="prismatic">
@@ -51,5 +51,5 @@
     <axis xyz = "0 1 0" />
     <origin rpy="0 0 0" xyz="0 -0.5 0"/>
-    <limit effort="1000.0" lower="-1" upper="1" velocity="0.5"/>
+    <limit effort="1000.0" lower="0" upper="1" velocity="0.5"/>
   </joint>
   <joint name="from_Y_to_end" type="fixed">

Commit message: created cell with 2 and 4 point robots and added dirrt pipeline

File: planar_cartesian_robot_description/urdf/cartesian_robot.urdf.xacro (robot description, xacro)
@@ -1,13 +1,4 @@
 <?xml version="1.0"?>
 <robot xmlns:xacro="http://ros.org/wiki/xacro" name="cartesian_robot" >
-  <material name="red">
-    <color rgba="0.8 0 0 1"/>
-  </material>
-  <material name="green">
-    <color rgba="0 0.8 0 1"/>
-  </material>
-  <material name="blue">
-    <color rgba="0 0 0.8 1"/>
-  </material>
   <material name="black">
     <color rgba="1 1 1 0.9"/>
